File: SMINIPROG.brd (EAGLE design)
At the start: 40 x 40 mm, 5 parts

Commit message: Routing for v1.0 release
Parts:
- added J1: ESPROG-SOCKET, SuperHouse-Connectors:ESPROG-S
- added J2: M01-PLAIN, SuperHouse-Connectors:1X01
- added TP6, TP7: POGO-P75-B1, SuperHouse-Test:PIN-1.02
- moved TP2 8.48 mm to (18.8, 38.7)
- moved TP4 5.76 mm to (20.2, 33.7)
- moved TP3 5.53 mm to (20.4, 35.5)
- moved TP1 4.47 mm to (19.0, 37.0)
- moved TP5 4.33 mm to (22.1, 26.4)
Connections:
- new net !RESET: J1.6, TP7.P$1
- new net 3.3V: J1.3, TP1.P$1
- new net GPIO0: J1.2, TP5.P$1
- new net GPIO2: J2.1, TP6.P$1
- new net SONOFF_RX: J1.4, TP4.P$1
- new net SONOFF_TX: J1.5, TP3.P$1
- net GND: now also J1.1
Routing:
- net GPIO2: track 0.00 -> 25.9 mm
- net SONOFF_RX: track 0.00 -> 19.0 mm
- net SONOFF_TX: track 0.00 -> 18.1 mm
- net GPIO0: track 0.00 -> 14.1 mm
- net !RESET: track 0.00 -> 11.1 mm
- added copper zone on layer 16, net 3.3V
- added copper zone on layer 1, net GND
- removed copper zone on layer 16, net GND
- removed copper zone on layer 1, net PAD
Other:
- board text added: "!RST"
- board text added: "3.3V"
- board text added: "Copyright 2019 SuperHouse Automation Pty Ltd Released under the terms of the TAPR Open Hardware Licence: tapr.org/OHL"
- board text added: "ESProg Header"
- board text added: "GND"
- board text added: "GPIO0"
- board text added: "GPIO2"
- board text added: "RX"
- board text added: "Sonoff Mini Programming Jig"
- board text added: "TX"
- board text added: "by Jon Oxer"
- board text added: "superhouse.tv/sminiprog"
- board text added: "v1.0"
- board text removed: "20mm v1.0"
- board text removed: "Sub-Mini Microswitch Breakout"
- board text removed: "superhouse.tv/smmb"

Commit message: Replaced ESP-Prog header, major update for v2.0 release
Parts:
- J1: value ESPROG-SOCKET -> ESP-PROG-1X6-2.54-SOCKET-RA; device SuperHouse-Connectors:ESPROG-S -> SuperHouse-ESP-Prog:1X6-2.54-SOCKET-RA
- moved J1 7.07 mm to (31.0, 20.0), turned to 270 degrees
Connections:
- net !RESET: now also J1.5; no longer J1.6
- net 3.3V: now also J1.4; no longer J1.3
- net GPIO0: now also J1.6; no longer J1.2
- net SONOFF_RX: now also J1.3; no longer J1.4
- net SONOFF_TX: now also J1.2; no longer J1.5
Routing:
- net !RESET: track 11.1 -> 24.8 mm
- net GPIO0: track 14.1 -> 16.4 mm
Other:
- board text added: "ESPFlasher Header"
- board text added: "v2.0"
- board text removed: "ESProg Header"
- board text removed: "v1.0"
